Commit message: fix bugs. 1. no xacro.py anymore, use xacro instead. 2.xacro marro usage: create:<xacro:macro name="mm".../> use:<xacro::mm .../>

File: urdf_demo/mybot_description/xacro/macros.xacro (robot description, xacro)
@@ -1,21 +1,21 @@
 <?xml version="1.0"?>
 <robot name="mybot" xmlns:xacro="http://www.ros.org/wiki/xacro">
-<macro name="cylinder_inertia" params="m r h">
+<xacro:macro name="cylinder_inertia" params="m r h">
   <inertia  ixx="${m*(3*r*r+h*h)/12}" ixy = "0" ixz = "0"
     iyy="${m*(3*r*r+h*h)/12}" iyz = "0"
     izz="${m*r*r/2}"
   />
-</macro>
-<macro name="box_inertia" params="m x y z">
+</xacro:macro>
+<xacro:macro name="box_inertia" params="m x y z">
   <inertia  ixx="${m*(y*y+z*z)/12}" ixy = "0" ixz = "0"
     iyy="${m*(x*x+z*z)/12}" iyz = "0"
     izz="${m*(x*x+z*z)/12}"
   />
-</macro>
-<macro name="sphere_inertia" params="m r">
+</xacro:macro>
+<xacro:macro name="sphere_inertia" params="m r">
   <inertia  ixx="${2*m*r*r/5}" ixy = "0" ixz = "0"
     iyy="${2*m*r*r/5}" iyz = "0"
     izz="${2*m*r*r/5}"
   />
-</macro>
+</xacro:macro>
 </robot>

File: urdf_demo/mybot_description/xacro/mybot.xacro (robot description, xacro)
@@ -40,5 +40,5 @@
     <origin xyz="0 0 ${wheelRadius}" rpy="0 0 0"/>
     <mass value="${chassisMass}"/>
-    <box_inertia m="${chassisMass}" x="${chassisLength}" y="${chassisWidth}" z="${chassisHeight}"/>
+    <xacro:box_inertia m="${chassisMass}" x="${chassisLength}" y="${chassisWidth}" z="${chassisHeight}"/>
   </inertial>
 </link>
@@ -64,5 +64,5 @@
     <origin xyz="${casterRadius-chassisLength/2} 0 ${casterRadius-chassisHeight+wheelRadius}" rpy="0 0 0"/>
     <mass value="${casterMass}"/>
-    <sphere_inertia m="${casterMass}" r="${casterRadius}"/>
+    <xacro:sphere_inertia m="${casterMass}" r="${casterRadius}"/>
   </inertial>
 </link>
@@ -84,5 +84,5 @@
     <origin xyz="0 0 0" rpy="0 ${PI/2} ${PI/2}" />
     <mass value="${wheelMass}"/>
-    <cylinder_inertia m="${wheelMass}" r="${wheelRadius}" h="${wheelWidth}"/>
+    <xacro:cylinder_inertia m="${wheelMass}" r="${wheelRadius}" h="${wheelWidth}"/>
   </inertial>
 </link>
@@ -122,5 +122,5 @@
     <origin xyz="0 0 0" rpy="0 ${PI/2} ${PI/2}" />
     <mass value="${wheelMass}"/>
-    <cylinder_inertia m="${wheelMass}" r="${wheelRadius}" h="${wheelWidth}"/>
+    <xacro:cylinder_inertia m="${wheelMass}" r="${wheelRadius}" h="${wheelWidth}"/>
   </inertial>
 </link>
